File: piec_oszust/piec_oszust.kicad_pcb (KiCad board)
At the start: 2 copper layers, 21 parts, among them J1 Jack-DC, J2 Conn_01x02_Pin, J3 PWM_IN, J4 Conn_01x02_Pin, Q1 BC547, Q2 BC547, U1 LM7805_TO220, U2 LM7808_TO220, U3 LM324

Commit message: updates, gerber, drill, map files added
Parts:
- J2: value Conn_01x02_Pin -> OUT_TRANSISTOR
- J4: value Conn_01x02_Pin -> OUT_OPAMP
- moved R8 30.3 mm to (80.0, 71.1)
- moved R9 30.0 mm to (72.4, 73.7)
- moved J2 29.3 mm to (95.2, 74.3), turned to -90 degrees
- moved R1 28.0 mm to (92.7, 61.0), turned to -90 degrees
- moved J3 27.9 mm to (71.1, 53.3), turned to 180 degrees
- moved R4 26.2 mm to (80.0, 82.5)
- moved R3 25.4 mm to (87.6, 80.0)
- moved Q1 21.3 mm to (85.1, 72.4), turned to 0 degrees
- moved Q2 18.7 mm to (93.1, 81.3), turned to 90 degrees
- moved C2 17.8 mm to (44.3, 57.1), turned to 180 degrees
- moved C1 17.7 mm to (38.2, 94.0), turned to 0 degrees
- moved R2 14.0 mm to (87.6, 77.5)
- moved A1 11.7 mm to (67.3, 91.4)
- moved U2 11.4 mm to (39.4, 66.0)
- moved U3 8.98 mm to (88.9, 61.0), turned to -90 degrees
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Connections:
- A1 pad 15: Net-(A1-D12) -> unconnected-(A1-D12-Pad15)
- R8 pad 1: Net-(A1-D12) -> Net-(R8-Pad1)
- R8 pad 2: Net-(J3-Pin_1) -> Net-(U3B--)
- R9 pad 2: Net-(A1-D12) -> Net-(R8-Pad1)
- U2 pad 2: unconnected-(U2-GND-Pad2) -> GND
- U3 pad 5: unconnected-(U3B-+-Pad5) -> Net-(J3-Pin_1)
- U3 pad 6: unconnected-(U3B---Pad6) -> Net-(U3B--)
- U3 pad 7: unconnected-(U3-Pad7) -> Net-(U3B--)
Routing:
- net +8V: track 0.00 -> 134.0 mm
- net +5V: track 0.00 -> 56.8 mm
- net D10: track 0.00 -> 31.7 mm
- net PWM_OUT_100_1: track 0.00 -> 25.3 mm
- net +12V: track 0.00 -> 22.2 mm
- net Net-(Q1-C): track 0.00 -> 13.4 mm
- net Net-(R5-Pad2): track 0.00 -> 13.0 mm
- net Net-(J3-Pin_1): track 0.00 -> 11.5 mm
- net Net-(U3B--): track 0.00 -> 10.7 mm
- net PWM_OUT_100_2: track 0.00 -> 10.5 mm
- net Net-(Q1-B): track 0.00 -> 9.40 mm
- net Net-(U3A--): track 0.00 -> 5.08 mm
- net Net-(R8-Pad1): track 0.00 -> 2.54 mm
- net GND: track 0.00 -> 0.90 mm
- added copper zone on B.Cu, net GND
Other:
- board outline added: 69.9 x 54.6 mm
- board text added: "PIEC TEST 2024"

Commit message: missing connection
Connections:
- A1 pad 15: unconnected-(A1-D12-Pad15) -> Net-(A1-D12)
- R8 pad 1: Net-(R8-Pad1) -> Net-(A1-D12)
- R9 pad 2: Net-(R8-Pad1) -> Net-(A1-D12)
Routing:
- net Net-(A1-D12): track 0.00 -> 28.2 mm
- net Net-(R8-Pad1): track 2.54 -> 0.00 mm
