File: piec_oszust/piec_oszust.kicad_sch (KiCad schematic)
At the start: 21 parts, among them J1 Jack-DC, J2 Conn_01x02_Pin, J3 PWM_IN, J4 Conn_01x02_Pin, Q1 BC547, Q2 BC547, U1 LM7805_TO220, U2 LM7808_TO220, U3 LM324

Commit message: updates, gerber, drill, map files added
Parts:
- J2: value Conn_01x02_Pin -> OUT_TRANSISTOR
- J4: value Conn_01x02_Pin -> OUT_OPAMP
Connections:
- net GND: now also U2.2 (GND)
- net at R8.1, R9.2: no longer A1.15 (D12)
- net at J3.1 (Pin_1): now also U3.5 (+); no longer R8.2
- net at U3.6 (-): now also R8.2, U3.7
Other:
- moved on the sheet: J3, R8, R9, U3B

Commit message: missing connection
Connections:
- net at A1.15 (D12): now also R8.1, R9.2
Changed lines of the file:
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@@
   (junction (at 162.56 57.15) (diameter 0) (color 0 0 0 0)
+  )
+  (junction (at 66.04 99.06) (diameter 0) (color 0 0 0 0)
   )
   (junction (at 176.53 68.58) (diameter 0) (color 0 0 0 0)
@@
     (stroke (width 0) (type default))
   )
+  (wire (pts (xy 66.04 99.06) (xy 76.2 99.06))
+    (stroke (width 0) (type default))
+  )
